File: electronics/climate_sensor_laundry.kicad_sch (KiCad schematic)
At the start: 31 parts, among them J1 Conn_01x04, J2 Conn_01x04, Q1 BS170, SW1 SW_Push, U1 NodeMCU1.0(ESP-12E), U2 display_i2c_1inch3, U3 DHT22, U4 DHT22

Commit message: works with external sensor over network
Parts:
- removed C? (x2): C, symbol Device:C
- removed J1, J2: Conn_01x04, Connector_JST:JST_XH_B4B-XH-AM_1x04_P2.50mm_Vertical, symbol Connector_Generic:Conn_01x04
- removed R5: 1k, Resistor_THT:R_Axial_DIN0204_L3.6mm_D1.6mm_P5.08mm_Horizontal, symbol Device:R
- removed U4: DHT22, Sensor:Aosong_DHT11_5.5x12.0_P2.54mm, symbol Sensor:DHT11
- removed U?: AMS1117-3.3, Package_TO_SOT_SMD:SOT-223-3_TabPin2, symbol Regulator_Linear:AMS1117-3.3
Connections:
- net dht_outside_2 is gone; now on net dht_outside_1: U1.26 (D4(GPIO2))
- net dht_outside_1: no longer U1.27 (D3(GPIO0))
- net ~{rst}: now reaches U1.13 (RST)
- net ~{rst}: now also U1.30 (D0(GPIO16))
- no-connect marks 13 -> 12
Other:
- company: (none) -> Gras7 Labs
- title: (none) -> Klimasensor Waschküche
- moved on the sheet: C?, J?, R4, R?, U3, U?
